File: front-board/iit_hawkrod_front_board.sch (EAGLE design)
At the start: 29 parts

Commit message: Add Status Lights
Parts:
- added STATUS_LIGHTS: 5-103635-3, 5-103635-3:5-103635-3
Connections:
- new net SIG_HRT_LED: STATUS_LIGHTS.4, U$6.13-SCK/LED
- net 5V: now also STATUS_LIGHTS.1
- net GND: now also STATUS_LIGHTS.2, STATUS_LIGHTS.3
Other:
- note added: "HRT_LED_3.3V"
- note added: "HRT_LED_GND"
- note added: "PWR_LED_5V"
- note added: "PWR_LED_GND"
Changed lines of the file:
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@@
 <part name="R_WHEEL_SENSOR" library="5-103635-2" deviceset="5-103635-2" device=""/>
 <part name="GND5" library="supply1" library_urn="urn:adsk.eagle:library:371" deviceset="GND" device=""/>
+<part name="STATUS_LIGHTS" library="5-103635-3" deviceset="5-103635-3" device=""/>
+<part name="GND6" library="supply1" library_urn="urn:adsk.eagle:library:371" deviceset="GND" device=""/>
 </parts>
 <sheets>
@@
 <text x="-2.032" y="-74.168" size="0.6096" layer="91">R_WHEEL_SENSE</text>
 <text x="-25.4" y="71.12" size="6.4516" layer="91">External I/O</text>
-<text x="127" y="-111.76" size="6.4516" layer="91">HawkRod 22'</text>
-<text x="127" y="-116.84" size="2.54" layer="91">Revision 2022.1-beta | Last Updated: 9/5/2022</text>
-<text x="127" y="-144.78" size="2.54" layer="91">Electrical Lead: Isaias Rivera
+<text x="127" y="-134.62" size="6.4516" layer="91">HawkRod 22'</text>
+<text x="127" y="-139.7" size="2.54" layer="91">Revision 2022.1-beta | Last Updated: 9/5/2022</text>
+<text x="127" y="-167.64" size="2.54" layer="91">Electrical Lead: Isaias Rivera
 Schematic designed by: Noah Husby
 PCB designed by: Hazim Zainedin</text>
+<text x="4.064" y="-160.274" size="0.6096" layer="91" rot="MR0">PWR_LED_GND</text>
+<text x="4.064" y="-162.814" size="0.6096" layer="91" rot="MR0">HRT_LED_GND</text>
+<text x="4.318" y="-157.734" size="0.6096" layer="91" rot="MR0">PWR_LED_5V</text>
+<text x="4.064" y="-165.354" size="0.6096" layer="91" rot="MR0">HRT_LED_3.3V</text>
 </plain>
 <instances>
@@
 <instance part="GND5" gate="1" x="27.94" y="-68.58" smashed="yes" rot="R180">
 <attribute name="VALUE" x="30.48" y="-66.04" size="1.778" layer="96" rot="R180"/>
+</instance>
+<instance part="STATUS_LIGHTS" gate="G$1" x="2.54" y="-160.02" smashed="yes" rot="MR0">
+<attribute name="NAME" x="7.6286" y="-154.29531875" size="1.781009375" layer="95" rot="MR0"/>
+<attribute name="VALUE" x="7.620140625" y="-170.1803" size="1.77805" layer="96" rot="MR0"/>
+</instance>
+<instance part="GND6" gate="1" x="27.94" y="-157.48" smashed="yes" rot="R180">
+<attribute name="VALUE" x="30.48" y="-154.94" size="1.778" layer="96" rot="R180"/>
 </instance>
 </instances>
@@
 <pinref part="GND5" gate="1" pin="GND"/>
 </segment>
+<segment>
+<wire x1="12.7" y1="-160.02" x2="27.94" y2="-160.02" width="0.1524" layer="91"/>
+<pinref part="GND6" gate="1" pin="GND"/>
+<pinref part="STATUS_LIGHTS" gate="G$1" pin="2"/>
+<pinref part="STATUS_LIGHTS" gate="G$1" pin="3"/>
+<wire x1="12.7" y1="-160.02" x2="12.7" y2="-162.56" width="0.1524" layer="91"/>
+<junction x="12.7" y="-160.02"/>
+</segment>
 </net>
 <net name="SIG_START_BUTTON" class="0">
@@
 <wire x1="12.7" y1="-68.58" x2="15.24" y2="-68.58" width="0.1524" layer="91"/>
 <label x="15.24" y="-68.58" size="1.27" layer="95" xref="yes"/>
+</segment>
+<segment>
+<wire x1="12.7" y1="-157.48" x2="15.24" y2="-157.48" width="0.1524" layer="91"/>
+<label x="15.24" y="-157.48" size="1.778" layer="95" rot="MR180" xref="yes"/>
+<pinref part="STATUS_LIGHTS" gate="G$1" pin="1"/>
 </segment>
 </net>
@@
 <pinref part="U$2" gate="G$1" pin="D"/>
 <wire x1="60.96" y1="-86.36" x2="60.96" y2="-81.28" width="0.1524" layer="91"/>
-<wire x1="60.96" y1="-81.28" x2="15.24" y2="-81.28" width="0.1524" layer="91"/>
-<wire x1="15.24" y1="-81.28" x2="15.24" y2="-93.98" width="0.1524" layer="91"/>
-<wire x1="15.24" y1="-93.98" x2="12.7" y2="-93.98" width="0.1524" layer="91"/>
+<wire x1="60.96" y1="-81.28" x2="12.7" y2="-81.28" width="0.1524" layer="91"/>
+<wire x1="12.7" y1="-81.28" x2="12.7" y2="-93.98" width="0.1524" layer="91"/>
 <pinref part="FAULT_INDICATORS" gate="G$1" pin="1"/>
 </segment>
@@
 <segment>
 <wire x1="116.84" y1="68.58" x2="-25.4" y2="68.58" width="0.1524" layer="91"/>
-<wire x1="116.84" y1="68.58" x2="116.84" y2="-149.86" width="0.1524" layer="91"/>
-<wire x1="116.84" y1="-149.86" x2="-25.4" y2="-149.86" width="0.1524" layer="91"/>
-<wire x1="-25.4" y1="-149.86" x2="-25.4" y2="68.58" width="0.1524" layer="91"/>
+<wire x1="116.84" y1="68.58" x2="116.84" y2="-172.72" width="0.1524" layer="91"/>
+<wire x1="116.84" y1="-172.72" x2="-25.4" y2="-172.72" width="0.1524" layer="91"/>
+<wire x1="-25.4" y1="-172.72" x2="-25.4" y2="68.58" width="0.1524" layer="91"/>
 </segment>
 </net>
 <net name="N$12" class="0">
 <segment>
-<wire x1="121.92" y1="-149.86" x2="121.92" y2="-99.06" width="0.1524" layer="91"/>
-<wire x1="121.92" y1="-99.06" x2="233.68" y2="-99.06" width="0.1524" layer="91"/>
-<wire x1="233.68" y1="-99.06" x2="233.68" y2="-149.86" width="0.1524" layer="91"/>
-<wire x1="233.68" y1="-149.86" x2="121.92" y2="-149.86" width="0.1524" layer="91"/>
-</segment>
-</net>
+<wire x1="121.92" y1="-172.72" x2="121.92" y2="-121.92" width="0.1524" layer="91"/>
+<wire x1="121.92" y1="-121.92" x2="233.68" y2="-121.92" width="0.1524" layer="91"/>
+<wire x1="233.68" y1="-121.92" x2="233.68" y2="-172.72" width="0.1524" layer="91"/>
+<wire x1="233.68" y1="-172.72" x2="121.92" y2="-172.72" width="0.1524" layer="91"/>
+</segment>
+</net>
+<net name="SIG_HRT_LED" class="0">
+<segment>
+<wire x1="203.2" y1="0" x2="205.74" y2="0" width="0.1524" layer="91"/>
+<label x="205.74" y="0" size="1.27" layer="95" xref="yes"/>
+<pinref part="U$6" gate="G$1" pin="13-SCK/LED"/>
+</segment>
+<segment>
+<wire x1="12.7" y1="-165.1" x2="15.24" y2="-165.1" width="0.1524" layer="91"/>
+<label x="15.24" y="-165.1" size="1.27" layer="95" xref="yes"/>
+<pinref part="STATUS_LIGHTS" gate="G$1" pin="4"/>
+</segment>
+</net>

Commit message: Add USB
Parts:
- added DASH_USB: 1-292303-1, 1-292303-1:1-292303-1
Connections:
- new net N$13: DASH_USB.3, U$6.D-
- new net N$16: DASH_USB.2, U$6.D+
- net 5V: now also DASH_USB.4
- net GND: now also DASH_USB.1, DASH_USB.SHIELD
Changed lines of the file:
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@@
 <part name="STATUS_LIGHTS" library="5-103635-3" deviceset="5-103635-3" device=""/>
 <part name="GND6" library="supply1" library_urn="urn:adsk.eagle:library:371" deviceset="GND" device=""/>
+<part name="DASH_USB" library="1-292303-1" deviceset="1-292303-1" device=""/>
+<part name="GND14" library="supply1" library_urn="urn:adsk.eagle:library:371" deviceset="GND" device=""/>
+<part name="GND16" library="supply1" library_urn="urn:adsk.eagle:library:371" deviceset="GND" device=""/>
 </parts>
 <sheets>
@@
 <attribute name="VALUE" x="30.48" y="-154.94" size="1.778" layer="96" rot="R180"/>
 </instance>
+<instance part="DASH_USB" gate="G$1" x="243.84" y="53.34" smashed="yes" rot="MR0">
+<attribute name="NAME" x="249.17691875" y="61.47245" size="1.77896875" layer="95" rot="MR0"/>
+<attribute name="VALUE" x="249.435990625" y="43.41983125" size="1.780540625" layer="96" rot="MR0"/>
+</instance>
+<instance part="GND14" gate="1" x="228.6" y="60.96" smashed="yes" rot="R180">
+<attribute name="VALUE" x="231.14" y="63.5" size="1.778" layer="96" rot="R180"/>
+</instance>
+<instance part="GND16" gate="1" x="228.6" y="45.72" smashed="yes" rot="R180">
+<attribute name="VALUE" x="231.14" y="48.26" size="1.778" layer="96" rot="R180"/>
+</instance>
 </instances>
 <busses>
@@
 <junction x="12.7" y="-160.02"/>
 </segment>
+<segment>
+<pinref part="GND14" gate="1" pin="GND"/>
+<pinref part="DASH_USB" gate="G$1" pin="1"/>
+<wire x1="228.6" y1="58.42" x2="233.68" y2="58.42" width="0.1524" layer="91"/>
+</segment>
+<segment>
+<pinref part="GND16" gate="1" pin="GND"/>
+<wire x1="228.6" y1="43.18" x2="233.68" y2="43.18" width="0.1524" layer="91"/>
+<pinref part="DASH_USB" gate="G$1" pin="SHIELD"/>
+<wire x1="233.68" y1="48.26" x2="233.68" y2="43.18" width="0.1524" layer="91"/>
+</segment>
 </net>
 <net name="SIG_START_BUTTON" class="0">
@@
 <label x="15.24" y="-157.48" size="1.778" layer="95" rot="MR180" xref="yes"/>
 <pinref part="STATUS_LIGHTS" gate="G$1" pin="1"/>
+</segment>
+<segment>
+<wire x1="233.68" y1="50.8" x2="231.14" y2="50.8" width="0.1524" layer="91"/>
+<label x="231.14" y="50.8" size="1.778" layer="95" rot="R180" xref="yes"/>
+<pinref part="DASH_USB" gate="G$1" pin="4"/>
 </segment>
 </net>
@@
 </segment>
 </net>
+<net name="N$13" class="0">
+<segment>
+<pinref part="U$6" gate="G$1" pin="D-"/>
+<wire x1="203.2" y1="45.72" x2="215.9" y2="45.72" width="0.1524" layer="91"/>
+<wire x1="215.9" y1="45.72" x2="215.9" y2="53.34" width="0.1524" layer="91"/>
+<pinref part="DASH_USB" gate="G$1" pin="3"/>
+<wire x1="215.9" y1="53.34" x2="233.68" y2="53.34" width="0.1524" layer="91"/>
+</segment>
+</net>
+<net name="N$16" class="0">
+<segment>
+<pinref part="U$6" gate="G$1" pin="D+"/>
+<wire x1="203.2" y1="43.18" x2="223.52" y2="43.18" width="0.1524" layer="91"/>
+<wire x1="223.52" y1="43.18" x2="223.52" y2="55.88" width="0.1524" layer="91"/>
+<pinref part="DASH_USB" gate="G$1" pin="2"/>
+<wire x1="223.52" y1="55.88" x2="233.68" y2="55.88" width="0.1524" layer="91"/>
+</segment>
+</net>

Commit message: Layout_Pre
Changed lines of the file:
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@@
 </instance>
 <instance part="R10" gate="G$1" x="81.28" y="-33.02" smashed="yes" rot="R90">
-<attribute name="NAME" x="79.7814" y="-36.83" size="1.778" layer="95" rot="R90"/>
+<attribute name="NAME" x="87.4014" y="-36.83" size="1.778" layer="95" rot="R90"/>
 <attribute name="VALUE" x="84.582" y="-36.83" size="1.778" layer="96" rot="R90"/>
 </instance>
 <instance part="R14" gate="G$1" x="76.2" y="-35.56" smashed="yes" rot="R90">
-<attribute name="NAME" x="74.7014" y="-39.37" size="1.778" layer="95" rot="R90"/>
+<attribute name="NAME" x="74.7014" y="-41.91" size="1.778" layer="95" rot="R90"/>
 <attribute name="VALUE" x="79.502" y="-39.37" size="1.778" layer="96" rot="R90"/>
 </instance>
